Commit message: fix: validate sim backend for so101 and axol

File: fm_control/urdf/axol.sim.urdf.xacro (robot description, xacro)
@@ -8,6 +8,7 @@
 variant is nominal; both arms are always emitted.
 Args:
-  sim_backend   mock | mujoco | gazebo | isaac  (selects the System plugin; no
-                real backend yet — Axol's CAN driver is deferred)
+  sim_backend   mock | mujoco | gz | gazebo | isaac  (selects the System plugin;
+                gz is an alias for gazebo; no real backend yet, as Axol's CAN
+                driver is deferred, so real fails the xacro like any unknown value)
   mujoco_model  MJCF the mujoco backend loads; injected by the fm_bringup registry
                 from fm_sim_models when sim_backend=mujoco (empty default otherwise)
@@ -15,4 +16,9 @@
 <robot xmlns:xacro="http://www.ros.org/wiki/xacro" name="axol">
   <xacro:arg name="sim_backend" default="mock"/>
+  <!-- Sets `backend`: gz becomes gazebo, and an unknown value fails the xacro. -->
+  <xacro:include filename="$(find fm_control)/urdf/sim_backend.xacro"/>
+  <xacro:fm_sim_backend
+      requested="$(arg sim_backend)"
+      supported="${['mock', 'mujoco', 'gazebo', 'isaac']}"/>
   <xacro:arg name="isaac_joint_commands_topic" default="/isaac_joint_commands"/>
   <xacro:arg name="isaac_joint_states_topic" default="/isaac_joint_states"/>
@@ -35,15 +41,15 @@
   <xacro:property name="left_elbow_ready" value="1.0"/>
   <xacro:property name="right_elbow_ready" value="-1.0"/>
-  <xacro:if value="${'$(arg sim_backend)' in single_system_backends}">
+  <xacro:if value="${backend in single_system_backends}">
     <xacro:axol_single_system
-        sim_backend="$(arg sim_backend)"
+        sim_backend="${backend}"
         left_elbow_ready="${left_elbow_ready}"
         right_elbow_ready="${right_elbow_ready}"
         mujoco_model_path="${mujoco_model_path}"/>
   </xacro:if>
-  <xacro:unless value="${'$(arg sim_backend)' in single_system_backends}">
+  <xacro:unless value="${backend in single_system_backends}">
     <xacro:axol_arm_system
         prefix="left_"
-        sim_backend="$(arg sim_backend)"
+        sim_backend="${backend}"
         elbow_ready="${left_elbow_ready}"
         mujoco_model_path="${mujoco_model_path}"
@@ -52,5 +58,5 @@
     <xacro:axol_arm_system
         prefix="right_"
-        sim_backend="$(arg sim_backend)"
+        sim_backend="${backend}"
         elbow_ready="${right_elbow_ready}"
         mujoco_model_path="${mujoco_model_path}"
@@ -60,5 +66,5 @@
   <!-- Gazebo hosts the controller_manager inside the sim via this world plugin,
        which loads the controllers.yaml. Emitted only for the gazebo backend. -->
-  <xacro:if value="${'$(arg sim_backend)' == 'gazebo'}">
+  <xacro:if value="${backend == 'gazebo'}">
     <gazebo>
       <plugin filename="gz_ros2_control-system"

File: fm_control/urdf/g1.sim.urdf.xacro (robot description, xacro)
@@ -13,5 +13,6 @@
 robot_state_publisher still serves TF + visuals.
 Args:
-  sim_backend   mock | mujoco | gazebo | isaac | real
+  sim_backend   mock | mujoco | gz | gazebo | isaac | real  (gz is an alias for
+                gazebo, anything else fails the xacro)
   mujoco_model  MJCF the mujoco backend loads; injected by the fm_bringup registry
                 from fm_sim_models when sim_backend=mujoco (empty default otherwise).
@@ -21,4 +22,9 @@
 <robot xmlns:xacro="http://www.ros.org/wiki/xacro" name="G1_D">
   <xacro:arg name="sim_backend" default="mock"/>
+  <!-- Sets `backend`: gz becomes gazebo, and an unknown value fails the xacro. -->
+  <xacro:include filename="$(find fm_control)/urdf/sim_backend.xacro"/>
+  <xacro:fm_sim_backend
+      requested="$(arg sim_backend)"
+      supported="${['mock', 'mujoco', 'gazebo', 'isaac', 'real']}"/>
   <xacro:arg name="isaac_joint_commands_topic" default="/isaac_joint_commands"/>
   <xacro:arg name="isaac_joint_states_topic" default="/isaac_joint_states"/>
@@ -35,5 +41,5 @@
   <xacro:include filename="$(find fm_control)/urdf/g1.ros2_control.xacro"/>
   <xacro:g1_system
-      sim_backend="$(arg sim_backend)"
+      sim_backend="${backend}"
       mujoco_model_path="${mujoco_model_path}"
       isaac_joint_commands_topic="$(arg isaac_joint_commands_topic)"
@@ -41,5 +47,5 @@
   <!-- Gazebo hosts the controller_manager inside the sim via this world plugin,
        which loads the controllers.yaml. Emitted only for the gazebo backend. -->
-  <xacro:if value="${'$(arg sim_backend)' == 'gazebo'}">
+  <xacro:if value="${backend == 'gazebo'}">
     <gazebo>
       <plugin filename="gz_ros2_control-system"

File: fm_control/urdf/openarm.sim.urdf.xacro (robot description, xacro)
@@ -18,13 +18,9 @@
   <xacro:arg name="robot_preset" default="right_arm"/>
   <xacro:arg name="sim_backend" default="mock"/>
-  <!-- gz is the simulation stack's name for Gazebo; the macros below say gazebo. -->
-  <xacro:property name="requested_backend" value="$(arg sim_backend)"/>
-  <xacro:property name="backend" value="${'gazebo' if requested_backend == 'gz' else requested_backend}"/>
-  <!-- An unknown value would otherwise emit a system with no <hardware>, which only
-       fails later inside controller_manager. -->
-  <xacro:if value="${backend not in ['mock', 'mujoco', 'gazebo', 'isaac', 'real']}">
-    ${xacro.fatal('unknown sim_backend: ' + str(requested_backend)
-                  + ' (expected mock, mujoco, gz, gazebo, isaac or real)')}
-  </xacro:if>
+  <!-- Sets `backend`: gz becomes gazebo, and an unknown value fails the xacro. -->
+  <xacro:include filename="$(find fm_control)/urdf/sim_backend.xacro"/>
+  <xacro:fm_sim_backend
+      requested="$(arg sim_backend)"
+      supported="${['mock', 'mujoco', 'gazebo', 'isaac', 'real']}"/>
   <xacro:arg name="collapse_internal_empty_links" default="true"/>
   <xacro:arg name="emit_grasp_frame" default="false"/>

File: fm_control/urdf/so101.sim.urdf.xacro (robot description, xacro)
@@ -7,5 +7,6 @@
 unlike the OpenArm, the variant is purely nominal.
 Args:
-  sim_backend   mock | mujoco | gazebo | isaac | real  (selects the System plugin)
+  sim_backend   mock | mujoco | gz | gazebo | isaac | real  (selects the System
+                plugin; gz is an alias for gazebo, anything else fails the xacro)
   usb_port      serial device for the real (feetech) backend; ignored by sim backends
   mujoco_model  MJCF the mujoco backend loads; injected by the fm_bringup registry
@@ -14,4 +15,9 @@
 <robot xmlns:xacro="http://www.ros.org/wiki/xacro" name="so101">
   <xacro:arg name="sim_backend" default="mock"/>
+  <!-- Sets `backend`: gz becomes gazebo, and an unknown value fails the xacro. -->
+  <xacro:include filename="$(find fm_control)/urdf/sim_backend.xacro"/>
+  <xacro:fm_sim_backend
+      requested="$(arg sim_backend)"
+      supported="${['mock', 'mujoco', 'gazebo', 'isaac', 'real']}"/>
   <xacro:arg name="usb_port" default="/dev/ttyACM0"/>
   <xacro:arg name="isaac_joint_commands_topic" default="/isaac_joint_commands"/>
@@ -29,5 +35,5 @@
   <xacro:include filename="$(find fm_control)/urdf/so101.ros2_control.xacro"/>
   <xacro:so101_arm_system
-      sim_backend="$(arg sim_backend)"
+      sim_backend="${backend}"
       usb_port="$(arg usb_port)"
       mujoco_model_path="${mujoco_model_path}"
@@ -36,5 +42,5 @@
   <!-- Gazebo hosts the controller_manager inside the sim via this world plugin,
        which loads the controllers.yaml. Emitted only for the gazebo backend. -->
-  <xacro:if value="${'$(arg sim_backend)' == 'gazebo'}">
+  <xacro:if value="${backend == 'gazebo'}">
     <gazebo>
       <plugin filename="gz_ros2_control-system"
