Commit message: feat: add openarm camera mounts and gz backend alias

File: fm_control/urdf/openarm.sim.urdf.xacro (robot description, xacro)
@@ -9,5 +9,6 @@
 Args:
   robot_preset   openarm_description v2.0 preset (right_arm, default_bimanual, ...)
-  sim_backend    mock | mujoco | gazebo | isaac | real  (selects the System plugin)
+  sim_backend    mock | mujoco | gz | gazebo | isaac | real  (selects the System
+                 plugin; gz is an alias for gazebo, anything else fails the xacro)
   can_interface  SocketCAN device for the real backend (ignored by sim backends)
   can_fd         CAN-FD toggle for the real backend
@@ -17,4 +18,13 @@
   <xacro:arg name="robot_preset" default="right_arm"/>
   <xacro:arg name="sim_backend" default="mock"/>
+  <!-- gz is the simulation stack's name for Gazebo; the macros below say gazebo. -->
+  <xacro:property name="requested_backend" value="$(arg sim_backend)"/>
+  <xacro:property name="backend" value="${'gazebo' if requested_backend == 'gz' else requested_backend}"/>
+  <!-- An unknown value would otherwise emit a system with no <hardware>, which only
+       fails later inside controller_manager. -->
+  <xacro:if value="${backend not in ['mock', 'mujoco', 'gazebo', 'isaac', 'real']}">
+    ${xacro.fatal('unknown sim_backend: ' + str(requested_backend)
+                  + ' (expected mock, mujoco, gz, gazebo, isaac or real)')}
+  </xacro:if>
   <xacro:arg name="collapse_internal_empty_links" default="true"/>
   <xacro:arg name="emit_grasp_frame" default="false"/>
@@ -34,4 +44,5 @@
   <xacro:include filename="$(find openarm_description)/assets/robot/openarm_v2.0/urdf/utils/openarm_v20_robot.xacro"/>
   <xacro:include filename="$(find fm_control)/urdf/openarm.ros2_control.xacro"/>
+  <xacro:include filename="$(find fm_description)/urdf/openarm_cameras.xacro"/>
   <xacro:property name="robot_root" value="$(find openarm_description)/assets/robot/openarm_v2.0"/>
   <xacro:property name="config_root" value="${robot_root + '/config'}"/>
@@ -80,5 +91,5 @@
       arm_specs="${arm_specs}"
       index="0"
-      sim_backend="$(arg sim_backend)"
+      sim_backend="${backend}"
       control_gains="${control_gains}"
       can_interface="$(arg can_interface)"
@@ -86,7 +97,14 @@
       isaac_joint_commands_topic="$(arg isaac_joint_commands_topic)"
       isaac_joint_states_topic="$(arg isaac_joint_states_topic)"/>
+  <!-- Camera frames on whichever links this preset carries. -->
+  <xacro:property name="right_arms" value="${[s for s in arm_specs if s['prefix'] == 'openarm_right_']}"/>
+  <xacro:openarm_cameras
+      body="${'body' in components and preset_cfg['body']['enabled']}"
+      right_arm="${len(right_arms) > 0}"
+      right_hand="${len(right_arms) > 0 and right_arms[0]['hand']}"
+      collapse_empty_links="$(arg collapse_internal_empty_links)"/>
   <!-- Gazebo hosts the controller_manager inside the sim via this world plugin,
        which loads the controllers.yaml. Emitted only for the gazebo backend. -->
-  <xacro:if value="${'$(arg sim_backend)' == 'gazebo'}">
+  <xacro:if value="${backend == 'gazebo'}">
     <gazebo>
       <plugin filename="gz_ros2_control-system"

Commit message: feat: add loader hand preset for sim openarm

File: fm_control/urdf/openarm.sim.urdf.xacro (robot description, xacro)
@@ -9,4 +9,11 @@
 Args:
   robot_preset   openarm_description v2.0 preset (right_arm, default_bimanual, ...)
+  hand           loader | pinch  (default loader). loader is the arm fm-rob-01's loader
+                 runs: its parallel-jaw hand (prismatic fingers, 0..0.05 m, grasp_frame
+                 0.18 m out) and its joint limits, from fm_description's loader
+                 variant of robot_preset. pinch is openarm_description's stock preset
+                 with the v2.0 pinch gripper. right_arm and left_arm carry no gripper,
+                 so they stay stock under either value; a gripper preset with no
+                 loader variant fails under loader. Only default_bimanual has one.
   sim_backend    mock | mujoco | gz | gazebo | isaac | real  (selects the System
                  plugin; gz is an alias for gazebo, anything else fails the xacro)
@@ -17,4 +24,5 @@
 <robot xmlns:xacro="http://www.ros.org/wiki/xacro" name="openarm_v20">
   <xacro:arg name="robot_preset" default="right_arm"/>
+  <xacro:arg name="hand" default="loader"/>
   <xacro:arg name="sim_backend" default="mock"/>
   <!-- Sets `backend`: gz becomes gazebo, and an unknown value fails the xacro. -->
@@ -41,8 +49,34 @@
   <xacro:include filename="$(find fm_control)/urdf/openarm.ros2_control.xacro"/>
   <xacro:include filename="$(find fm_description)/urdf/openarm_cameras.xacro"/>
+  <xacro:include filename="$(find fm_description)/urdf/openarm_parallel_hand.xacro"/>
   <xacro:property name="robot_root" value="$(find openarm_description)/assets/robot/openarm_v2.0"/>
   <xacro:property name="config_root" value="${robot_root + '/config'}"/>
+  <!-- The preset name becomes a file path, so it must be a plain name. -->
+  <xacro:property name="preset_name" value="$(arg robot_preset)"/>
+  <xacro:unless value="${preset_name[:1].isalpha() and preset_name.isascii()
+                         and preset_name.replace('_', '').isalnum()}">
+    ${xacro.fatal('invalid robot_preset: ' + repr(preset_name))}
+  </xacro:unless>
+  <!-- `hand` is the arg as given; `loader_hand` below is whether the loader hand is
+       built. An arm spec's `hand` key says only that the arm has some gripper. -->
+  <xacro:property name="hand" value="$(arg hand)"/>
+  <xacro:unless value="${hand in ['loader', 'pinch']}">
+    ${xacro.fatal('unknown hand: ' + str(hand) + ' (expected loader or pinch)')}
+  </xacro:unless>
+  <xacro:property name="stock_cfg"
+      value="${xacro.load_yaml(config_root + '/robot_presets/' + preset_name + '.yaml')}"/>
+  <!-- Presets fm_description has a loader variant of, under config/openarm/loader_presets. -->
+  <xacro:property name="loader_presets" value="${['default_bimanual']}"/>
+  <xacro:property name="loader_hand" value="${hand == 'loader' and preset_name in loader_presets}"/>
+  <xacro:if value="${hand == 'loader' and not loader_hand
+                     and len([n for n in stock_cfg['robot']['components']
+                              if stock_cfg[n]['type'] == 'end_effector'
+                              and stock_cfg[n]['enabled']]) > 0}">
+    ${xacro.fatal('robot_preset ' + preset_name + ' has no loader-hand variant'
+                  + ' (one of ' + ', '.join(loader_presets) + '); pass hand:=pinch')}
+  </xacro:if>
   <xacro:property name="preset_cfg"
-      value="${xacro.load_yaml(config_root + '/robot_presets/' + '$(arg robot_preset)' + '.yaml')}"/>
+      value="${xacro.load_yaml('$(find fm_description)/config/openarm/loader_presets/'
+                               + preset_name + '.yaml') if loader_hand else stock_cfg}"/>
   <!-- Emit links + joints for the preset. -->
   <xacro:openarm_v20_robot
@@ -52,6 +86,6 @@
       emit_grasp_frame="$(arg emit_grasp_frame)"/>
   <!-- Resolve one spec per enabled arm: its prefix and whether it carries a gripper
-       (an enabled end_effector attached to it). Iteration order follows the preset's
-       robot.components, so joint order matches the geometry. -->
+       (the loader hand, or an enabled end_effector attached to it). Iteration order
+       follows the preset's robot.components, so joint order matches the geometry. -->
   <xacro:property name="components" value="${preset_cfg['robot']['components']}"/>
   <xacro:property name="arm_names"
@@ -75,5 +109,5 @@
                             * (ready_bimanual if len(arm_names) > 1 else ready_single)[i]
                             for i in python.range(7)],
-                     hand=len([m for m in components
+                     hand=loader_hand or len([m for m in components
                                if preset_cfg[m]['type'] == 'end_effector'
                                and preset_cfg[m]['enabled']
@@ -82,4 +116,17 @@
                                and preset_cfg[m]['connection']['attach_to'] == n]) > 0)
                 for n in arm_names]}"/>
+  <!-- The loader hand on every arm, one arm per call. -->
+  <xacro:macro name="openarm_parallel_hands" params="arm_specs index">
+    <xacro:if value="${index &lt; len(arm_specs)}">
+      <xacro:openarm_parallel_hand
+          prefix="${arm_specs[index]['prefix']}"
+          flange="${arm_specs[index]['prefix']}link7"
+          emit_grasp_frame="$(arg emit_grasp_frame)"/>
+      <xacro:openarm_parallel_hands arm_specs="${arm_specs}" index="${index + 1}"/>
+    </xacro:if>
+  </xacro:macro>
+  <xacro:if value="${loader_hand}">
+    <xacro:openarm_parallel_hands arm_specs="${arm_specs}" index="0"/>
+  </xacro:if>
   <xacro:property name="single_system_backends" value="${['mujoco', 'gazebo']}"/>
   <!-- Control gains feed the real backend only; loaded once and passed through. -->
@@ -109,4 +156,5 @@
       right_arm="${len(right_arms) > 0}"
       right_hand="${len(right_arms) > 0 and right_arms[0]['hand']}"
+      loader_hand="${loader_hand}"
       collapse_empty_links="$(arg collapse_internal_empty_links)"/>
   <!-- Gazebo hosts the controller_manager inside the sim via this world plugin,

File: fm_description/urdf/openarm_cameras.xacro (robot description, xacro)
@@ -10,13 +10,16 @@
   cam_wrist_r_optical        ->   openarm_right_cam_wrist_optical
   parent follower_body_link0 ->   openarm_body_link0  (same frame)
-  parent follower_r_hand     ->   openarm_right_cam_wrist_mount  (same frame)
+  parent follower_r_hand     ->   openarm_right_hand, or openarm_right_cam_wrist_mount
+                                 at the same frame when the arm has no loader hand
 Args:
   body                  the preset enables the body (the chest camera's parent)
   right_arm             the preset enables the right arm (the wrist camera's)
   right_hand            the right arm carries a gripper
+  loader_hand           the gripper is the loader hand (openarm_parallel_hand.xacro),
+                        which carries the hand frame itself
   collapse_empty_links  collapse_internal_empty_links was passed to openarm_description
 -->
 <robot xmlns:xacro="http://www.ros.org/wiki/xacro">
-  <xacro:macro name="openarm_cameras" params="body right_arm right_hand collapse_empty_links">
+  <xacro:macro name="openarm_cameras" params="body right_arm right_hand loader_hand collapse_empty_links">
     <!-- Chest camera (UVC fisheye). First calibrated on fm-rob-01 on 2026-10-01 by the
          classical baseline's calibrate_chest: an ArUco marker on the right wrist bracket
@@ -39,11 +42,12 @@
       </joint>
     </xacro:if>
-    <xacro:if value="${right_arm}">
+    <!-- The loader hand is Anvil's follower_r_hand, which the wrist pose was measured
+         against. Without it, openarm_right_cam_wrist_mount stands in at the same frame. -->
+    <xacro:if value="${right_arm and not loader_hand}">
       <!-- With a gripper and collapsed empty links, openarm_description folds link7
            into ee_base_link, which keeps link7's frame. -->
       <xacro:property name="right_wrist_parent"
           value="${'openarm_right_ee_base_link' if right_hand and collapse_empty_links else 'openarm_right_link7'}"/>
-      <!-- Anvil's follower_r_hand frame, which the wrist pose was measured against.
-           Anvil and openarm_description share every joint axis and link7 frame, but
+      <!-- Anvil and openarm_description share every joint axis and link7 frame, but
            Anvil's hand sits 100.1 mm out along the wrist and flipped about x. -->
       <link name="openarm_right_cam_wrist_mount"/>
@@ -53,4 +57,6 @@
         <origin xyz="0 0 -0.1001" rpy="${pi} 0 0"/>
       </joint>
+    </xacro:if>
+    <xacro:if value="${right_arm}">
       <!-- Right wrist camera. From Anvil's CAD URDF (right_wrist_cam_joint on
            right_hand). On recorded wrist frames, with the chest camera's intrinsics
@@ -60,5 +66,5 @@
       <link name="openarm_right_cam_wrist_optical"/>
       <joint name="openarm_right_cam_wrist_optical_joint" type="fixed">
-        <parent link="openarm_right_cam_wrist_mount"/>
+        <parent link="${'openarm_right_hand' if loader_hand else 'openarm_right_cam_wrist_mount'}"/>
         <child link="openarm_right_cam_wrist_optical"/>
         <origin xyz="0.074 0.001 0.009" rpy="-0.8255 0.0 1.5708"/>

Commit message: fix: add loader wrist and clear ready pose

File: fm_control/urdf/openarm.sim.urdf.xacro (robot description, xacro)
@@ -101,9 +101,17 @@
        `ready` is the RIGHT-arm spawn joint vector: for a bimanual preset (2+ arms) a
        "hands forward, ~20cm apart" pre-grasp pose so the 1:1 mirror's engage baseline matches
-       a natural two-hand start; for a single arm the original splayed bent-ready pose. -->
-  <xacro:property name="ready_bimanual" value="${[0.6816, 0.0265, -0.3161, 1.1622, 0.0, 0.3, 0.0]}"/>
+       a natural two-hand start; for a single arm the original splayed bent-ready pose.
+       The loader hands are 168 mm wide and touch at the pinch pose, so the loader's
+       bimanual pose spreads joint2 to 0.13 rad: the grasp frames sit 210 mm apart and
+       the hands keep 53 mm clear with the fingers fully open (test_openarm_loader_hand
+       checks it on the collision meshes). -->
+  <xacro:property name="ready_bimanual_pinch" value="${[0.6816, 0.0265, -0.3161, 1.1622, 0.0, 0.3, 0.0]}"/>
+  <xacro:property name="ready_bimanual_loader" value="${[0.6816, 0.13, -0.3161, 1.1622, 0.0, 0.3, 0.0]}"/>
+  <xacro:property name="ready_bimanual"
+      value="${ready_bimanual_loader if loader_hand else ready_bimanual_pinch}"/>
   <xacro:property name="ready_single" value="${[0.0, 0.5, 0.0, 1.2, 0.0, 0.3, 0.0]}"/>
   <xacro:property name="arm_specs"
       value="${[dict(prefix=preset_cfg[n]['prefix'],
+                     mirror=preset_cfg[n].get('reflect', dict()).get('y', 1),
                      ready=[(preset_cfg[n].get('reflect', dict()).get('y', 1) if i != 3 else 1)
                             * (ready_bimanual if len(arm_names) > 1 else ready_single)[i]
@@ -122,4 +130,5 @@
           prefix="${arm_specs[index]['prefix']}"
           flange="${arm_specs[index]['prefix']}link7"
+          mirror="${arm_specs[index]['mirror']}"
           emit_grasp_frame="$(arg emit_grasp_frame)"/>
       <xacro:openarm_parallel_hands arm_specs="${arm_specs}" index="${index + 1}"/>

File: fm_description/urdf/openarm_parallel_hand.xacro (robot description, xacro)
@@ -10,5 +10,6 @@
 hence the large z offsets.
   snapshot (follower_r_*)        here (<prefix> = openarm_right_)
-  link7 (flange)            ->   <prefix>ee_base_link, fixed at link7's frame
+  link7 (flange)            ->   <prefix>ee_base_link, fixed at link7's frame, with
+                                 link7's v1.0 wrist mesh and inertial
   hand                      ->   <prefix>hand: ee_base_link + (0, 0, -0.1001), rpy (pi, 0, 0)
   hand_tcp                  ->   <prefix>grasp_frame: hand + (0, 0, 0.08), approach +z
@@ -18,7 +19,15 @@
 hand pose, written from link7 as (0, 0, 0.1001), rpy (0, 0, pi/2), is the same frame
 as the one above. Both arms use the same pose.
+openarm_description v2.0 leaves link7 bare and puts the wrist on its end effector,
+so with no v2.0 end effector the loader's link7 geometry and its 0.466 kg go on
+ee_base_link. The loader's link7 frame is ee_base_link turned half a turn about
+(1, mirror, 0): rpy (pi, 0, mirror * pi/2). The mesh (openarm_description's
+openarm_v1.0 link7) sits at (0, 0, -0.5585) in that frame, (0, 0, 0.5585) here; the
+inertial is the loader's, rotated into ee_base_link. fm-sim's patched OpenArm MJCF
+carries the same numbers, so every backend has the same wrist.
 Args:
   prefix            arm prefix, e.g. openarm_right_
   flange            the link joint7 drives (the arm's link7)
+  mirror            the arm's reflect on y: 1 for the right arm, -1 for the left
   emit_grasp_frame  add <prefix>grasp_frame, the robot profile's ee_frame
 -->
@@ -26,20 +35,27 @@
   <xacro:property name="parallel_hand_meshes"
       value="package://openarm_description/assets/end_effector/parallel_link/meshes"/>
-  <!-- Visual and collision share an origin and mesh. scale_y -1 mirrors the finger mesh. -->
-  <xacro:macro name="openarm_parallel_hand_geometry" params="name mesh xyz scale_y:=1">
+  <xacro:property name="v1_arm_meshes"
+      value="package://openarm_description/assets/robot/openarm_v1.0/mesh/arm"/>
+  <!-- Visual and collision share an origin. scale_y -1 mirrors the mesh. -->
+  <xacro:macro name="openarm_mesh_geometry"
+      params="name visual collision xyz rpy:='0 0 0' scale_y:=1">
     <visual name="${name}_visual">
-      <origin xyz="${xyz}" rpy="0 0 0"/>
+      <origin xyz="${xyz}" rpy="${rpy}"/>
       <geometry>
-        <mesh filename="${parallel_hand_meshes}/visual/${mesh}.dae"
-              scale="0.001 ${0.001 * scale_y} 0.001"/>
+        <mesh filename="${visual}" scale="0.001 ${0.001 * scale_y} 0.001"/>
       </geometry>
     </visual>
     <collision name="${name}_collision">
-      <origin xyz="${xyz}" rpy="0 0 0"/>
+      <origin xyz="${xyz}" rpy="${rpy}"/>
       <geometry>
-        <mesh filename="${parallel_hand_meshes}/collision/${mesh}.stl"
-              scale="0.001 ${0.001 * scale_y} 0.001"/>
+        <mesh filename="${collision}" scale="0.001 ${0.001 * scale_y} 0.001"/>
       </geometry>
     </collision>
+  </xacro:macro>
+  <xacro:macro name="openarm_parallel_hand_geometry" params="name mesh xyz scale_y:=1">
+    <xacro:openarm_mesh_geometry
+        name="${name}" xyz="${xyz}" scale_y="${scale_y}"
+        visual="${parallel_hand_meshes}/visual/${mesh}.dae"
+        collision="${parallel_hand_meshes}/collision/${mesh}.stl"/>
   </xacro:macro>
   <!-- One finger link and its prismatic joint. side_sign is -1 for the right finger
@@ -67,7 +83,22 @@
     </joint>
   </xacro:macro>
-  <xacro:macro name="openarm_parallel_hand" params="prefix flange emit_grasp_frame">
-    <!-- The pinch preset's flange name, so the arm ends in the same link either way. -->
-    <link name="${prefix}ee_base_link"/>
+  <xacro:macro name="openarm_parallel_hand" params="prefix flange mirror emit_grasp_frame">
+    <!-- The pinch preset's flange name, so the arm ends in the same link either way.
+         It carries the loader's link7 wrist (see the header); the left arm's mesh
+         and inertial are the right's mirrored in y. -->
+    <link name="${prefix}ee_base_link">
+      <xacro:openarm_mesh_geometry
+          name="${prefix}link7" xyz="0 0 0.5585" rpy="${pi} 0 ${mirror * pi / 2}"
+          scale_y="${mirror}"
+          visual="${v1_arm_meshes}/visual/link7.dae"
+          collision="${v1_arm_meshes}/collision/link7_symp.stl"/>
+      <inertial>
+        <origin xyz="0.01266175250761268 ${mirror * 6.875510271106056e-05} -0.06951945409987448"
+                rpy="0 0 0"/>
+        <mass value="0.4659771327380578"/>
+        <inertia ixx="0.000497" ixy="${mirror * 1e-06}" ixz="-8.9e-05"
+                 iyy="0.000639" iyz="${mirror * -1e-06}" izz="0.000342"/>
+      </inertial>
+    </link>
     <joint name="${prefix}ee_base_joint" type="fixed">
       <parent link="${flange}"/>
