Commit message: feat: bimanual mirror spawn and ready poses for openarm

File: fm_control/urdf/openarm.ros2_control.xacro (robot description, xacro)
@@ -92,4 +92,5 @@
   <xacro:macro name="openarm_arm_system"
       params="prefix hand sim_backend control_gains
+              init1 init2 init3 init4 init5 init6 init7
               can_interface:=can0 can_fd:=true
               isaac_joint_commands_topic:=/isaac_joint_commands
@@ -108,12 +109,22 @@
            singularity) — MoveIt Servo then emergency-stops every cycle and refuses to
            jog (logs "close to a position limit. Halting" + "Very close to a singularity").
-           A bent elbow lifts it off both. initial_value is applied by the sim hardware. -->
-      <xacro:openarm_joint joint_name="${prefix}joint1"/>
-      <xacro:openarm_joint joint_name="${prefix}joint2" initial_position="0.5"/>
-      <xacro:openarm_joint joint_name="${prefix}joint3"/>
-      <xacro:openarm_joint joint_name="${prefix}joint4" initial_position="1.2"/>
-      <xacro:openarm_joint joint_name="${prefix}joint5"/>
-      <xacro:openarm_joint joint_name="${prefix}joint6" initial_position="0.3"/>
-      <xacro:openarm_joint joint_name="${prefix}joint7"/>
+           A bent elbow lifts it off both. initial_value is applied by the sim hardware.
+           `ready` is the RIGHT-arm ready joint vector (per preset, from openarm.sim.urdf.xacro):
+           the single-arm splayed pose, or the bimanual "hands forward, ~20cm apart" pre-grasp
+           pose (so the 1:1 mirror's engage baseline matches a natural two-hand start instead
+           of the arms being ~59cm apart). mirror_sign flips the reflected (left) arm's ready
+           pose so both arms spawn as sagittal mirror images: the left arm is the right reflected
+           about Y with joint AXES pointing the SAME world direction (the reflect macro mirrors
+           joint ORIGINS, not axes), so by the mirror identity M*R(a,q)*M = R(M*a,-q) the
+           reflected joints {1,2,3,5,6,7} need NEGATED angles; joint4 (excluded from the reflect)
+           keeps its sign. The per-joint initN are the FINAL (mirror-applied) spawn angles,
+           computed per arm in openarm.sim.urdf.xacro's arm_specs. -->
+      <xacro:openarm_joint joint_name="${prefix}joint1" initial_position="${init1}"/>
+      <xacro:openarm_joint joint_name="${prefix}joint2" initial_position="${init2}"/>
+      <xacro:openarm_joint joint_name="${prefix}joint3" initial_position="${init3}"/>
+      <xacro:openarm_joint joint_name="${prefix}joint4" initial_position="${init4}"/>
+      <xacro:openarm_joint joint_name="${prefix}joint5" initial_position="${init5}"/>
+      <xacro:openarm_joint joint_name="${prefix}joint6" initial_position="${init6}"/>
+      <xacro:openarm_joint joint_name="${prefix}joint7" initial_position="${init7}"/>
       <xacro:if value="${hand}">
         <xacro:openarm_joint joint_name="${prefix}finger_joint1"/>
@@ -131,4 +142,7 @@
           prefix="${spec['prefix']}"
           hand="${spec['hand']}"
+          init1="${spec['ready'][0]}" init2="${spec['ready'][1]}" init3="${spec['ready'][2]}"
+          init4="${spec['ready'][3]}" init5="${spec['ready'][4]}" init6="${spec['ready'][5]}"
+          init7="${spec['ready'][6]}"
           sim_backend="${sim_backend}"
           control_gains="${control_gains}"

File: fm_control/urdf/openarm.sim.urdf.xacro (robot description, xacro)
@@ -53,6 +53,18 @@
                 and preset_cfg[n]['config'] == 'arm'
                 and preset_cfg[n]['enabled']]}"/>
+  <!-- mirror_sign is the preset's sagittal reflect on Y (+1 for a base arm, -1 for the
+       mirrored arm). The left arm is the right reflected about the XZ plane, so equal joint
+       angles would tilt both arms the SAME world direction; the reflected joints must be
+       sign-flipped by mirror_sign to spawn as a true mirror. Applied in openarm_arm_system.
+       `ready` is the RIGHT-arm spawn joint vector: for a bimanual preset (2+ arms) a
+       "hands forward, ~20cm apart" pre-grasp pose so the 1:1 mirror's engage baseline matches
+       a natural two-hand start; for a single arm the original splayed bent-ready pose. -->
+  <xacro:property name="ready_bimanual" value="${[0.6816, 0.0265, -0.3161, 1.1622, 0.0, 0.3, 0.0]}"/>
+  <xacro:property name="ready_single" value="${[0.0, 0.5, 0.0, 1.2, 0.0, 0.3, 0.0]}"/>
   <xacro:property name="arm_specs"
       value="${[dict(prefix=preset_cfg[n]['prefix'],
+                     ready=[(preset_cfg[n].get('reflect', dict()).get('y', 1) if i != 3 else 1)
+                            * (ready_bimanual if len(arm_names) > 1 else ready_single)[i]
+                            for i in python.range(7)],
                      hand=len([m for m in components
                                if preset_cfg[m]['type'] == 'end_effector'

Commit message: fix: load one sim system for both openarm arms

File: fm_control/urdf/openarm.ros2_control.xacro (robot description, xacro)
@@ -2,7 +2,9 @@
 <!--
 First Motive backend-selectable ros2_control for the OpenArm.
-One <ros2_control> system per enabled arm. The controllers, controller_manager,
-and the command/state interface set stay identical across every backend — only the
-<hardware> System plugin swaps, selected by the `sim_backend` arg:
+One <ros2_control> system per enabled arm, except under mujoco and gazebo, which
+get a single system for every arm (openarm_single_system).
+The controllers, controller_manager, and the command/state interface set stay
+identical across every backend — only the <hardware> System plugin swaps, selected
+by the `sim_backend` arg:
   mock    -> mock_components/GenericSystem        (no sim; perfect state echo)
   mujoco  -> mujoco_ros2_control/MujocoSystemInterface  (Mac daily driver, CPU)
@@ -94,6 +96,37 @@
     </joint>
   </xacro:macro>
-  <!-- One <ros2_control> system for a single arm: backend hardware + 7 arm joints,
-       plus finger_joint1 when the arm carries a gripper. -->
+  <!-- One arm's joints: 7 arm joints, plus finger_joint1 when it carries a gripper.
+       Shared by the per-arm systems and the single system, so both emit the same
+       interfaces and spawn pose. -->
+  <xacro:macro name="openarm_arm_joints"
+      params="prefix hand init1 init2 init3 init4 init5 init6 init7">
+    <!-- Spawn in a bent "ready" pose, NOT all-zeros. joint4 (elbow) has lower limit
+         = 0, so a zeros spawn sits AT the joint limit AND fully extended (a kinematic
+         singularity) — MoveIt Servo then emergency-stops every cycle and refuses to
+         jog (logs "close to a position limit. Halting" + "Very close to a singularity").
+         A bent elbow lifts it off both. initial_value is applied by the sim hardware.
+         `ready` is the RIGHT-arm ready joint vector (per preset, from openarm.sim.urdf.xacro):
+         the single-arm splayed pose, or the bimanual "hands forward, ~20cm apart" pre-grasp
+         pose (so the 1:1 mirror's engage baseline matches a natural two-hand start instead
+         of the arms being ~59cm apart). mirror_sign flips the reflected (left) arm's ready
+         pose so both arms spawn as sagittal mirror images: the left arm is the right reflected
+         about Y with joint AXES pointing the SAME world direction (the reflect macro mirrors
+         joint ORIGINS, not axes), so by the mirror identity M*R(a,q)*M = R(M*a,-q) the
+         reflected joints {1,2,3,5,6,7} need NEGATED angles; joint4 (excluded from the reflect)
+         keeps its sign. The per-joint initN are the FINAL (mirror-applied) spawn angles,
+         computed per arm in openarm.sim.urdf.xacro's arm_specs. -->
+    <xacro:openarm_joint joint_name="${prefix}joint1" initial_position="${init1}"/>
+    <xacro:openarm_joint joint_name="${prefix}joint2" initial_position="${init2}"/>
+    <xacro:openarm_joint joint_name="${prefix}joint3" initial_position="${init3}"/>
+    <xacro:openarm_joint joint_name="${prefix}joint4" initial_position="${init4}"/>
+    <xacro:openarm_joint joint_name="${prefix}joint5" initial_position="${init5}"/>
+    <xacro:openarm_joint joint_name="${prefix}joint6" initial_position="${init6}"/>
+    <xacro:openarm_joint joint_name="${prefix}joint7" initial_position="${init7}"/>
+    <xacro:if value="${hand}">
+      <xacro:openarm_joint joint_name="${prefix}finger_joint1"/>
+    </xacro:if>
+  </xacro:macro>
+  <!-- One <ros2_control> system for a single arm: backend hardware + that arm's
+       joints. -->
   <xacro:macro name="openarm_arm_system"
       params="prefix hand sim_backend control_gains
@@ -111,29 +144,8 @@
           isaac_joint_commands_topic="${isaac_joint_commands_topic}"
           isaac_joint_states_topic="${isaac_joint_states_topic}" />
-      <!-- Spawn in a bent "ready" pose, NOT all-zeros. joint4 (elbow) has lower limit
-           = 0, so a zeros spawn sits AT the joint limit AND fully extended (a kinematic
-           singularity) — MoveIt Servo then emergency-stops every cycle and refuses to
-           jog (logs "close to a position limit. Halting" + "Very close to a singularity").
-           A bent elbow lifts it off both. initial_value is applied by the sim hardware.
-           `ready` is the RIGHT-arm ready joint vector (per preset, from openarm.sim.urdf.xacro):
-           the single-arm splayed pose, or the bimanual "hands forward, ~20cm apart" pre-grasp
-           pose (so the 1:1 mirror's engage baseline matches a natural two-hand start instead
-           of the arms being ~59cm apart). mirror_sign flips the reflected (left) arm's ready
-           pose so both arms spawn as sagittal mirror images: the left arm is the right reflected
-           about Y with joint AXES pointing the SAME world direction (the reflect macro mirrors
-           joint ORIGINS, not axes), so by the mirror identity M*R(a,q)*M = R(M*a,-q) the
-           reflected joints {1,2,3,5,6,7} need NEGATED angles; joint4 (excluded from the reflect)
-           keeps its sign. The per-joint initN are the FINAL (mirror-applied) spawn angles,
-           computed per arm in openarm.sim.urdf.xacro's arm_specs. -->
-      <xacro:openarm_joint joint_name="${prefix}joint1" initial_position="${init1}"/>
-      <xacro:openarm_joint joint_name="${prefix}joint2" initial_position="${init2}"/>
-      <xacro:openarm_joint joint_name="${prefix}joint3" initial_position="${init3}"/>
-      <xacro:openarm_joint joint_name="${prefix}joint4" initial_position="${init4}"/>
-      <xacro:openarm_joint joint_name="${prefix}joint5" initial_position="${init5}"/>
-      <xacro:openarm_joint joint_name="${prefix}joint6" initial_position="${init6}"/>
-      <xacro:openarm_joint joint_name="${prefix}joint7" initial_position="${init7}"/>
-      <xacro:if value="${hand}">
-        <xacro:openarm_joint joint_name="${prefix}finger_joint1"/>
-      </xacro:if>
+      <xacro:openarm_arm_joints
+          prefix="${prefix}" hand="${hand}"
+          init1="${init1}" init2="${init2}" init3="${init3}" init4="${init4}"
+          init5="${init5}" init6="${init6}" init7="${init7}"/>
     </ros2_control>
   </xacro:macro>
@@ -168,3 +180,37 @@
     </xacro:if>
   </xacro:macro>
+  <!-- Recurse over the arm specs, emitting each arm's joints into the system the
+       caller has open. -->
+  <xacro:macro name="openarm_emit_arm_joints" params="arm_specs index">
+    <xacro:if value="${index &lt; len(arm_specs)}">
+      <xacro:property name="spec" value="${arm_specs[index]}" lazy_eval="false"/>
+      <xacro:openarm_arm_joints
+          prefix="${spec['prefix']}"
+          hand="${spec['hand']}"
+          init1="${spec['ready'][0]}" init2="${spec['ready'][1]}" init3="${spec['ready'][2]}"
+          init4="${spec['ready'][3]}" init5="${spec['ready'][4]}" init6="${spec['ready'][5]}"
+          init7="${spec['ready'][6]}"/>
+      <xacro:openarm_emit_arm_joints arm_specs="${arm_specs}" index="${index + 1}"/>
+    </xacro:if>
+  </xacro:macro>
+  <!-- One <ros2_control> system holding every arm's joints, for the simulators.
+       Each MujocoSystemInterface loads its own copy of the MJCF, so per-arm systems
+       would step the arms in separate worlds where they cannot touch each other or
+       the scene; gz_ros2_control stalls at "Waiting RM to load and initialize
+       hardware" with two GazeboSimSystem systems and comes up with one. -->
+  <xacro:macro name="openarm_single_system" params="arm_specs sim_backend">
+    <ros2_control name="openarm_system" type="system">
+      <!-- Placeholder prefix, gains, CAN and isaac topics: the mujoco and gazebo
+           hardware read none of them. -->
+      <xacro:openarm_backend_hardware
+          prefix=""
+          sim_backend="${sim_backend}"
+          control_gains="${dict()}"
+          can_interface=""
+          can_fd="false"
+          isaac_joint_commands_topic=""
+          isaac_joint_states_topic="" />
+      <xacro:openarm_emit_arm_joints arm_specs="${arm_specs}" index="0"/>
+    </ros2_control>
+  </xacro:macro>
 </robot>

File: fm_control/urdf/openarm.sim.urdf.xacro (robot description, xacro)
@@ -67,5 +67,6 @@
        mirrored arm). The left arm is the right reflected about the XZ plane, so equal joint
        angles would tilt both arms the SAME world direction; the reflected joints must be
-       sign-flipped by mirror_sign to spawn as a true mirror. Applied in openarm_arm_system.
+       sign-flipped by mirror_sign to spawn as a true mirror. Applied in arm_specs below;
+       consumed by openarm_arm_joints.
        `ready` is the RIGHT-arm spawn joint vector: for a bimanual preset (2+ arms) a
        "hands forward, ~20cm apart" pre-grasp pose so the 1:1 mirror's engage baseline matches
@@ -85,16 +86,25 @@
                                and preset_cfg[m]['connection']['attach_to'] == n]) > 0)
                 for n in arm_names]}"/>
+  <xacro:property name="single_system_backends" value="${['mujoco', 'gazebo']}"/>
   <!-- Control gains feed the real backend only; loaded once and passed through. -->
   <xacro:property name="control_gains"
       value="${xacro.load_yaml(config_root + '/arm/control/control_gains.yaml')}"/>
-  <xacro:openarm_emit_arm_systems
-      arm_specs="${arm_specs}"
-      index="0"
-      sim_backend="${backend}"
-      control_gains="${control_gains}"
-      can_interface="$(arg can_interface)"
-      can_fd="$(arg can_fd)"
-      isaac_joint_commands_topic="$(arg isaac_joint_commands_topic)"
-      isaac_joint_states_topic="$(arg isaac_joint_states_topic)"/>
+  <!-- The simulators share one system across both arms: MuJoCo loads one MJCF world
+       per system, and gz_ros2_control never initialises its hardware with two. Every
+       other backend, real hardware included, keeps one system per arm. -->
+  <xacro:if value="${backend in single_system_backends}">
+    <xacro:openarm_single_system arm_specs="${arm_specs}" sim_backend="${backend}"/>
+  </xacro:if>
+  <xacro:unless value="${backend in single_system_backends}">
+    <xacro:openarm_emit_arm_systems
+        arm_specs="${arm_specs}"
+        index="0"
+        sim_backend="${backend}"
+        control_gains="${control_gains}"
+        can_interface="$(arg can_interface)"
+        can_fd="$(arg can_fd)"
+        isaac_joint_commands_topic="$(arg isaac_joint_commands_topic)"
+        isaac_joint_states_topic="$(arg isaac_joint_states_topic)"/>
+  </xacro:unless>
   <!-- Camera frames on whichever links this preset carries. -->
   <xacro:property name="right_arms" value="${[s for s in arm_specs if s['prefix'] == 'openarm_right_']}"/>

Commit message: fix: drive the openarm finger mimic under gazebo

File: fm_control/urdf/openarm.ros2_control.xacro (robot description, xacro)
@@ -5,6 +5,6 @@
 get a single system for every arm (openarm_single_system).
 The controllers, controller_manager, and the command/state interface set stay
-identical across every backend — only the <hardware> System plugin swaps, selected
-by the `sim_backend` arg:
+identical across every backend, except gazebo's extra finger_joint2 state (below) —
+only the <hardware> System plugin swaps, selected by the `sim_backend` arg:
   mock    -> mock_components/GenericSystem        (no sim; perfect state echo)
   mujoco  -> mujoco_ros2_control/MujocoSystemInterface  (Mac daily driver, CPU)
@@ -14,5 +14,7 @@
 Joint names mirror openarm_description geometry exactly: <prefix>joint1..7, plus
 <prefix>finger_joint1 when the arm carries a gripper. `prefix` is the preset's full
-arm prefix, e.g. openarm_right_.
+arm prefix, e.g. openarm_right_. Under gazebo the system also lists
+<prefix>finger_joint2, state only, so gz_ros2_control drives it as the mimic of
+finger_joint1; DART has no mimic constraint and the finger would not move.
 -->
 <robot xmlns:xacro="http://www.ros.org/wiki/xacro">
@@ -98,7 +100,8 @@
   <!-- One arm's joints: 7 arm joints, plus finger_joint1 when it carries a gripper.
        Shared by the per-arm systems and the single system, so both emit the same
-       interfaces and spawn pose. -->
+       interfaces and spawn pose. mimic_finger adds finger_joint2 with no command
+       interface, which ros2_control reads as the URDF <mimic> of finger_joint1. -->
   <xacro:macro name="openarm_arm_joints"
-      params="prefix hand init1 init2 init3 init4 init5 init6 init7">
+      params="prefix hand init1 init2 init3 init4 init5 init6 init7 mimic_finger:=false">
     <!-- Spawn in a bent "ready" pose, NOT all-zeros. joint4 (elbow) has lower limit
          = 0, so a zeros spawn sits AT the joint limit AND fully extended (a kinematic
@@ -125,4 +128,9 @@
     <xacro:if value="${hand}">
       <xacro:openarm_joint joint_name="${prefix}finger_joint1"/>
+      <xacro:if value="${mimic_finger}">
+        <joint name="${prefix}finger_joint2">
+          <state_interface name="position"/>
+        </joint>
+      </xacro:if>
     </xacro:if>
   </xacro:macro>
@@ -182,5 +190,5 @@
   <!-- Recurse over the arm specs, emitting each arm's joints into the system the
        caller has open. -->
-  <xacro:macro name="openarm_emit_arm_joints" params="arm_specs index">
+  <xacro:macro name="openarm_emit_arm_joints" params="arm_specs index mimic_finger:=false">
     <xacro:if value="${index &lt; len(arm_specs)}">
       <xacro:property name="spec" value="${arm_specs[index]}" lazy_eval="false"/>
@@ -190,6 +198,8 @@
           init1="${spec['ready'][0]}" init2="${spec['ready'][1]}" init3="${spec['ready'][2]}"
           init4="${spec['ready'][3]}" init5="${spec['ready'][4]}" init6="${spec['ready'][5]}"
-          init7="${spec['ready'][6]}"/>
-      <xacro:openarm_emit_arm_joints arm_specs="${arm_specs}" index="${index + 1}"/>
+          init7="${spec['ready'][6]}"
+          mimic_finger="${mimic_finger}"/>
+      <xacro:openarm_emit_arm_joints
+          arm_specs="${arm_specs}" index="${index + 1}" mimic_finger="${mimic_finger}"/>
     </xacro:if>
   </xacro:macro>
@@ -198,5 +208,7 @@
        would step the arms in separate worlds where they cannot touch each other or
        the scene; gz_ros2_control stalls at "Waiting RM to load and initialize
-       hardware" with two GazeboSimSystem systems and comes up with one. -->
+       hardware" with two GazeboSimSystem systems and comes up with one. MuJoCo
+       couples the fingers with an equality in the MJCF; Gazebo needs the mimic
+       joint listed here. -->
   <xacro:macro name="openarm_single_system" params="arm_specs sim_backend">
     <ros2_control name="openarm_system" type="system">
@@ -211,5 +223,6 @@
           isaac_joint_commands_topic=""
           isaac_joint_states_topic="" />
-      <xacro:openarm_emit_arm_joints arm_specs="${arm_specs}" index="0"/>
+      <xacro:openarm_emit_arm_joints
+          arm_specs="${arm_specs}" index="0" mimic_finger="${sim_backend == 'gazebo'}"/>
     </ros2_control>
   </xacro:macro>
